File: GammaDSB.sch (KiCad schematic (older format))
At the start: 75 parts, among them J1 AudioIn, J2 AudioOut, J3 Conn_Coaxial, J4 Barrel_Jack, K1 G5V-2, Q1 BC-817, Q2 BC-817, Q3 BC-817, Q4 BC-817, Q5 C1162, Q6 BC817, Q7 BC-817, Q8 BC-817, T1 FT37-43 BIF8T, U1 MCP1700-5002E_SOT89, U2 NE602, Y1 7074, Y2 7074

Commit message: Small improvements.
Parts:
- removed Q6: BC817, Package_TO_SOT_SMD:SOT-23, symbol Transistor_BJT:BC817
- added Q6: BC807, Package_TO_SOT_SMD:SOT-23, symbol Transistor_BJT:BC807
Connections:
- net +12V: now also R16.2, R19.2, R20.2
- net at C5.1, U2.1 (IN_A), Y1.1: no longer C10.2, C8.1, U2.2 (IN_B)
- net at R18.2: now also Q6.1 (B)
- net at D3.2 (A), R21.2: now also Q6.3 (C)
- net at C27.1, R20.1: now also Q6.2 (E)
- new net: C10.2, C8.1, U2.2 (IN_B)
Changed lines of the file:
@@
 EESchema Schematic File Version 4
+LIBS:GammaDSB-cache
 EELAYER 29 0
 EELAYER END
@@
 encoding utf-8
 Sheet 1 1
-Title ""
-Date ""
+Title "Gamma DSB Transceiver"
+Date "2021-01-26"
 Rev ""
 Comp ""
@@
 	2450 3500 2450 3150
 Wire Wire Line
-	2450 3500 2250 3500
-Wire Wire Line
 	2250 3500 2250 3150
-Connection ~ 2450 3500
 Wire Wire Line
 	2250 3500 2250 3550
@@
 Wire Wire Line
 	4275 4600 4275 4525
-$Comp
-L Transistor_BJT:BC817 Q6
-U 1 1 604FEFD7
-P 4525 5225
-F 0 "Q6" H 4716 5179 50  0000 L CNN
-F 1 "BC817" H 4716 5270 50  0000 L CNN
-F 2 "Package_TO_SOT_SMD:SOT-23" H 4725 5150 50  0001 L CIN
-F 3 "http://www.fairchildsemi.com/ds/BC/BC817.pdf" H 4525 5225 50  0001 L CNN
-	1    4525 5225
-	1    0    0    1
-$EndComp
 Wire Wire Line
 	4325 5225 4250 5225
@@
 	1150 7025 1375 7025
 Connection ~ 1375 7025
+$Comp
+L power:+12V #PWR0109
+U 1 1 601119AE
+P 4275 4175
+F 0 "#PWR0109" H 4275 4025 50  0001 C CNN
+F 1 "+12V" H 4290 4348 50  0000 C CNN
+F 2 "" H 4275 4175 50  0001 C CNN
+F 3 "" H 4275 4175 50  0001 C CNN
+	1    4275 4175
+	1    0    0    -1
+$EndComp
+$Comp
+L Transistor_BJT:BC807 Q6
+U 1 1 6011203F
+P 4525 5225
+F 0 "Q6" H 4716 5179 50  0000 L CNN
+F 1 "BC807" H 4716 5270 50  0000 L CNN
+F 2 "Package_TO_SOT_SMD:SOT-23" H 4725 5150 50  0001 L CIN
+F 3 "http://www.fairchildsemi.com/ds/BC/BC807.pdf" H 4525 5225 50  0001 L CNN
+	1    4525 5225
+	1    0    0    1
+$EndComp
 $EndSCHEMATC
