File: GammaDSB.sch (KiCad schematic (older format))
At the start: 77 parts, among them J1 AudioIn, J2 AudioOut, J3 Conn_Coaxial, J4 Barrel_Jack, J5 Conn_01x01, J6 Conn_01x01, J7 Conn_01x01, K1 G5V-2, Q1 BC-817, Q2 BC-817, Q3 BC-817, Q4 BC-817, Q5 C1162, Q6 BC807, Q7 BC-817, Q8 BC-817, U1 MCP1700-5002E_SOT89, U2 NE602, Y1 7074, Y2 7074

Commit message: Changed layout, removed filter, smaller PCB size.
Parts:
- removed C22, C24, C25: 100n, Capacitor_SMD:C_0603_1608Metric, symbol GammaDSB-rescue:C-Device
- removed L2, L3: L, Inductor_THT:L_Toroid_Vertical_L16.0mm_W8.0mm_P7.62mm, symbol GammaDSB-rescue:L-Device
- C1, C10, C11, C12, C13, C14, C15, C16, C17, C18, C19, C2, C20, C21, C26, C27, C28, C3, C4, C5, C6, C7, C8, C9: symbol GammaDSB-rescue:C-Device -> GammaDSB-rescue:C-Device-GammaDSB-rescue
- C23: symbol GammaDSB-rescue:CP-Device -> GammaDSB-rescue:CP-Device-GammaDSB-rescue
- D1, D2: symbol GammaDSB-rescue:LED-Device -> GammaDSB-rescue:LED-Device-GammaDSB-rescue
- D3: symbol GammaDSB-rescue:D-Device -> GammaDSB-rescue:D-Device-GammaDSB-rescue
- J1, J2: symbol GammaDSB-rescue:AudioJack2_Ground-Connector -> GammaDSB-rescue:AudioJack2_Ground-Connector-GammaDSB-rescue
- J3: symbol GammaDSB-rescue:Conn_Coaxial-Connector -> GammaDSB-rescue:Conn_Coaxial-Connector-GammaDSB-rescue
- J4: symbol Connector:Barrel_Jack -> GammaDSB-rescue:Barrel_Jack-Connector
- J5, J6, J7: footprint Connector_Pin:Pin_D1.3mm_L11.0mm -> Connector_Wire:SolderWirePad_1x01_Drill0.8mm; symbol Connector:Conn_01x01 -> GammaDSB-rescue:Conn_01x01-Connector
- K1: symbol GammaDSB-rescue:G5V-2-Relay -> GammaDSB-rescue:G5V-2-Relay-GammaDSB-rescue
- L1: symbol GammaDSB-rescue:L_Core_Ferrite-Device -> GammaDSB-rescue:L_Core_Ferrite-Device-GammaDSB-rescue
- Q1, Q2, Q3, Q4, Q7, Q8: symbol GammaDSB-rescue:Q_NPN_BEC-Device -> GammaDSB-rescue:Q_NPN_BEC-Device-GammaDSB-rescue
- Q5: symbol GammaDSB-rescue:Q_NPN_ECB-Device -> GammaDSB-rescue:Q_NPN_ECB-Device-GammaDSB-rescue
- Q6: symbol GammaDSB-rescue:BC807-Transistor_BJT -> GammaDSB-rescue:BC807-Transistor_BJT-GammaDSB-rescue
- R1, R10, R11, R12, R13, R14, R15, R16, R17, R18, R19, R2, R20, R21, R22, R23, R3, R4, R5, R6, R7, R8, R9: symbol GammaDSB-rescue:R-Device -> GammaDSB-rescue:R-Device-GammaDSB-rescue
- U1: symbol GammaDSB-rescue:MCP1700-5002E_SOT89-Regulator_Linear -> GammaDSB-rescue:MCP1700-5002E_SOT89-Regulator_Linear-GammaDSB-rescue
- U2: symbol GammaDSB-rescue:NE602-riske-symbols -> GammaDSB-rescue:NE602-riske-symbols-GammaDSB-rescue
- Y1, Y2: symbol GammaDSB-rescue:Crystal-Device -> GammaDSB-rescue:Crystal-Device-GammaDSB-rescue
Connections:
- net at K1.13: now also J3.1 (In)
Other:
- moved on the sheet: J3
